File: Enose_PCB.kicad_sch (KiCad schematic)
At the start: 10 parts

Commit message: added some connectors
Parts:
- added D?: ESDLC5V0PB8, Package_DFN_QFN:UDFN-9_1.0x3.8mm_P0.5mm, symbol Power_Protection:ESDLC5V0PB8
- added J?: DA15_Pins, symbol Connector:DA15_Pins
- added J? (x3): B4B-XH-A_LF__SN_, B4B-XH-A_LF__SN_:JST_B4B-XH-A_LF__SN_, symbol B4B-XH-A_LF__SN_:B4B-XH-A_LF__SN_
Connections:
- net GND: now also D?.3 (A), J?.13 (P13), J?.14 (P14), J?.5, J?.6
- new net +15V: J?.15 (P15), J?.7, J?.8
- new net PWM1: D?.1 (K1), J?.12 (P12)
- new net PWM2: D?.2 (K2), J?.4
- new net PWM3: D?.4 (K3), J?.11 (P111)
- new net PWM4: D?.5 (K4), J?.3
- new net PWM5: D?.6 (K5), J?.10 (P10)
- new net PWM6: D?.7 (K6), J?.2
- new net PWM7: D?.8 (K7), J?.9 (P9)
- new net PWM8: D?.9 (K8), J?.1
