File: Power.kicad_sch (KiCad schematic)
At the start: 54 parts

Commit message: added some connectors
Other:
- moved on the sheet: C?
Changed lines of the file:
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@@
 	(wire
 		(pts
+			(xy 52.07 109.22) (xy 52.07 110.49)
+		)
+		(stroke
+			(width 0)
+			(type default)
+		)
+	)
+	(wire
+		(pts
 			(xy 242.57 27.94) (xy 242.57 25.4)
 		)
@@
 	(wire
 		(pts
+			(xy 45.72 109.22) (xy 45.72 110.49)
+		)
+		(stroke
+			(width 0)
+			(type default)
+		)
+	)
+	(wire
+		(pts
 			(xy 163.83 25.4) (xy 166.37 25.4)
 		)
@@
 	(symbol
 		(lib_id "power:GND")
-		(at 52.07 102.87 180)
+		(at 52.07 101.6 180)
 		(unit 1)
 		(exclude_from_sim no)
@@
 		(fields_autoplaced yes)
 		(property "Reference" "#PWR048"
-			(at 52.07 96.52 0)
+			(at 52.07 95.25 0)
 			(effects
 				(font
@@
 		)
 		(property "Value" "GND"
-			(at 52.07 97.79 0)
+			(at 52.07 96.52 0)
 			(effects
 				(font
@@
 		)
 		(property "Footprint" ""
-			(at 52.07 102.87 0)
+			(at 52.07 101.6 0)
 			(effects
 				(font
@@
 		)
 		(property "Datasheet" ""
-			(at 52.07 102.87 0)
+			(at 52.07 101.6 0)
 			(effects
 				(font
@@
 		)
 		(property "Description" "Power symbol creates a global label with name \"GND\" , ground"
-			(at 52.07 102.87 0)
+			(at 52.07 101.6 0)
 			(effects
 				(font
@@
 	(symbol
 		(lib_id "Device:C")
-		(at 45.72 106.68 0)
+		(at 45.72 105.41 0)
 		(mirror y)
 		(unit 1)
@@
 		(dnp no)
 		(property "Reference" "C?"
-			(at 42.672 103.886 0)
+			(at 42.672 102.616 0)
 			(effects
 				(font
@@
 		)
 		(property "Value" "22uF"
-			(at 42.672 106.426 0)
+			(at 42.672 105.156 0)
 			(effects
 				(font
@@
 		)
 		(property "Footprint" ""
-			(at 44.7548 110.49 0)
+			(at 44.7548 109.22 0)
 			(effects
 				(font
@@
 		)
 		(property "Datasheet" "~"
-			(at 45.72 106.68 0)
+			(at 45.72 105.41 0)
 			(effects
 				(font
@@
 		)
 		(property "Description" "Unpolarized capacitor"
-			(at 45.72 106.68 0)
+			(at 45.72 105.41 0)
 			(effects
 				(font
@@
 	(symbol
 		(lib_id "Device:C")
-		(at 52.07 106.68 0)
+		(at 52.07 105.41 0)
 		(unit 1)
 		(exclude_from_sim no)
@@
 		(fields_autoplaced yes)
 		(property "Reference" "C?"
-			(at 55.88 105.4099 0)
+			(at 55.88 104.1399 0)
 			(effects
 				(font
@@
 		)
 		(property "Value" "22uF"
-			(at 55.88 107.9499 0)
+			(at 55.88 106.6799 0)
 			(effects
 				(font
@@
 		)
 		(property "Footprint" ""
-			(at 53.0352 110.49 0)
+			(at 53.0352 109.22 0)
 			(effects
 				(font
@@
 		)
 		(property "Datasheet" "~"
-			(at 52.07 106.68 0)
+			(at 52.07 105.41 0)
 			(effects
 				(font
@@
 		)
 		(property "Description" "Unpolarized capacitor"
-			(at 52.07 106.68 0)
+			(at 52.07 105.41 0)
 			(effects
 				(font
@@
 	(symbol
 		(lib_id "power:GND")
-		(at 45.72 102.87 180)
+		(at 45.72 101.6 180)
 		(unit 1)
 		(exclude_from_sim no)
@@
 		(fields_autoplaced yes)
 		(property "Reference" "#PWR047"
-			(at 45.72 96.52 0)
+			(at 45.72 95.25 0)
 			(effects
 				(font
@@
 		)
 		(property "Value" "GND"
-			(at 45.72 97.79 0)
+			(at 45.72 96.52 0)
 			(effects
 				(font
@@
 		)
 		(property "Footprint" ""
-			(at 45.72 102.87 0)
+			(at 45.72 101.6 0)
 			(effects
 				(font
@@
 		)
 		(property "Datasheet" ""
-			(at 45.72 102.87 0)
+			(at 45.72 101.6 0)
 			(effects
 				(font
@@
 		)
 		(property "Description" "Power symbol creates a global label with name \"GND\" , ground"
-			(at 45.72 102.87 0)
+			(at 45.72 101.6 0)
 			(effects
 				(font
