File: Enose_PCB/Enose_PCB.kicad_sch (KiCad schematic)
At the start: 15 parts

Commit message: Added footprints
Parts:
- gave numbers to parts that had none: 15
Changed lines of the file:
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@@
 		(dnp no)
 		(fields_autoplaced yes)
-		(property "Reference" "C?"
+		(property "Reference" "C1"
 			(at 36.83 26.6699 0)
 			(effects
@@
 			(project "Enose_PCB"
 				(path "/eef70be0-4107-491c-8ca0-465071a6397e"
-					(reference "C?")
+					(reference "C1")
 					(unit 1)
 				)
@@
 		(on_board yes)
 		(dnp no)
-		(property "Reference" "C?"
+		(property "Reference" "C2"
 			(at 58.42 16.256 90)
 			(effects
@@
 			(project ""
 				(path "/eef70be0-4107-491c-8ca0-465071a6397e"
-					(reference "C?")
+					(reference "C2")
 					(unit 1)
 				)
@@
 		(dnp no)
 		(fields_autoplaced yes)
-		(property "Reference" "J?"
+		(property "Reference" "J4"
 			(at 248.92 113.0299 0)
 			(effects
@@
 			(project ""
 				(path "/eef70be0-4107-491c-8ca0-465071a6397e"
-					(reference "J?")
+					(reference "J4")
 					(unit 1)
 				)
@@
 		(dnp no)
 		(fields_autoplaced yes)
-		(property "Reference" "D?"
+		(property "Reference" "D1"
 			(at 236.22 142.2399 0)
 			(effects
@@
 			(project ""
 				(path "/eef70be0-4107-491c-8ca0-465071a6397e"
-					(reference "D?")
+					(reference "D1")
 					(unit 1)
 				)
@@
 		(dnp no)
 		(fields_autoplaced yes)
-		(property "Reference" "R?"
+		(property "Reference" "R1"
 			(at 35.56 38.0999 0)
 			(effects
@@
 			(project ""
 				(path "/eef70be0-4107-491c-8ca0-465071a6397e"
-					(reference "R?")
+					(reference "R1")
 					(unit 1)
 				)
@@
 		(dnp no)
 		(fields_autoplaced yes)
-		(property "Reference" "SW?"
+		(property "Reference" "SW1"
 			(at 29.21 46.99 0)
 			(effects
@@
 			(project "Enose_PCB"
 				(path "/eef70be0-4107-491c-8ca0-465071a6397e"
-					(reference "SW?")
+					(reference "SW1")
 					(unit 1)
 				)
@@
 		(dnp no)
 		(fields_autoplaced yes)
-		(property "Reference" "J?"
+		(property "Reference" "J2"
 			(at 247.65 50.7999 0)
 			(effects
@@
 			(project ""
 				(path "/eef70be0-4107-491c-8ca0-465071a6397e"
-					(reference "J?")
+					(reference "J2")
 					(unit 1)
 				)
@@
 		(dnp no)
 		(fields_autoplaced yes)
-		(property "Reference" "J?"
+		(property "Reference" "J1"
 			(at 247.65 34.2899 0)
 			(effects
@@
 			(project ""
 				(path "/eef70be0-4107-491c-8ca0-465071a6397e"
-					(reference "J?")
+					(reference "J1")
 					(unit 1)
 				)
@@
 		(dnp no)
 		(fields_autoplaced yes)
-		(property "Reference" "SW?"
+		(property "Reference" "SW2"
 			(at 120.65 46.9899 90)
 			(effects
@@
 			(project "Enose_PCB"
 				(path "/eef70be0-4107-491c-8ca0-465071a6397e"
-					(reference "SW?")
+					(reference "SW2")
 					(unit 1)
 				)
@@
 		(on_board yes)
 		(dnp no)
-		(property "Reference" "C?"
+		(property "Reference" "C3"
 			(at 58.674 34.29 90)
 			(effects
@@
 			(project ""
 				(path "/eef70be0-4107-491c-8ca0-465071a6397e"
-					(reference "C?")
+					(reference "C3")
 					(unit 1)
 				)
@@
 		(dnp no)
 		(fields_autoplaced yes)
-		(property "Reference" "U?"
+		(property "Reference" "U1"
 			(at 55.5341 38.1 0)
 			(effects
@@
 			(project "Enose_PCB"
 				(path "/eef70be0-4107-491c-8ca0-465071a6397e"
-					(reference "U?")
+					(reference "U1")
 					(unit 1)
 				)
@@
 		(dnp no)
 		(fields_autoplaced yes)
-		(property "Reference" "J?"
+		(property "Reference" "J3"
 			(at 247.65 67.3099 0)
 			(effects
@@
 			(project ""
 				(path "/eef70be0-4107-491c-8ca0-465071a6397e"
-					(reference "J?")
+					(reference "J3")
 					(unit 1)
 				)
@@
 		(dnp no)
 		(fields_autoplaced yes)
-		(property "Reference" "R?"
+		(property "Reference" "R3"
 			(at 121.92 33.0199 0)
 			(effects
@@
 			(project "Enose_PCB"
 				(path "/eef70be0-4107-491c-8ca0-465071a6397e"
-					(reference "R?")
+					(reference "R3")
 					(unit 1)
 				)
@@
 		(dnp no)
 		(fields_autoplaced yes)
-		(property "Reference" "R?"
+		(property "Reference" "R2"
 			(at 87.63 39.3699 0)
 			(effects
@@
 			(project "Enose_PCB"
 				(path "/eef70be0-4107-491c-8ca0-465071a6397e"
-					(reference "R?")
+					(reference "R2")
 					(unit 1)
 				)
@@
 		(dnp no)
 		(fields_autoplaced yes)
-		(property "Reference" "C?"
+		(property "Reference" "C4"
 			(at 138.43 48.2599 0)
 			(effects
@@
 			(project "Enose_PCB"
 				(path "/eef70be0-4107-491c-8ca0-465071a6397e"
-					(reference "C?")
-					(unit 1)
-				)
+					(reference "C4")
+					(unit 1)
+				)
