File: Enose_PCB/Power.kicad_sch (KiCad schematic)
At the start: 54 parts

Commit message: Added footprints
Parts:
- removed C?: 22uF, symbol Device:C
- C10: renamed from C?; footprint (none) -> Capacitor_SMD:C_0805_2012Metric
- J5: renamed from J?; footprint (none) -> Connector_USB:USB_C_Receptacle_GCT_USB4105-xx-A_16P_TopMnt_Horizontal
- L1: renamed from L?; footprint (none) -> SRP4030FA-1R0M:SRP4030FA1R0M
- L2: renamed from L?; footprint (none) -> SRP5030CA-1R0M:INDPM5355X310N
- L3: renamed from L?; value 3.5uH -> 4.7uH; footprint (none) -> Inductor_SMD:L_Coilcraft_XAL6060-XXX
- gave numbers to parts that had none: 48
Other:
- note added: "Uncertainties: - Signal ground - Loop Stability (is using example okay?) - NTC Filter - USB data to Battery charger - Too high output capcitance??"
- note removed: "Uncertainties: - Signal ground - Loop Stability (is using example okay?) - NTC Filter - USB data to Battery charger - Buck-Boost converter values - USB Connecter Pin count - Too high output capcitance?? - No/few low capacitance capacitors"
- moved on the sheet: C23, TP4
