File: Enose_PCB/cellular.module.kicad_sch (KiCad schematic)
At the start: 44 parts

Commit message: Added footprints
Parts:
- removed C? (x3): NC, symbol Device:C
- removed J?: SIM_Card, symbol Connector:SIM_Card
- removed Q? (x4): Q_NPN, symbol Device:Q_NPN
- added J9: 2229333-2, 22293332, symbol 2229333-2:2229333-2
- added Q2, Q3, Q4, Q5: Q_NPN, MMBT3904LT1G:SOT96P237X111-3N, symbol Device:Q_NPN
- Q1: renamed from Q?; footprint (none) -> MMBT3904LT1G:SOT96P237X111-3N
- gave numbers to parts that had none: 35
Connections:
- net GND: now also J9.10 (GND_4), J9.11 (GND_5), J9.12 (GND_6), J9.13 (GND_7), J9.14 (GND_8), J9.15 (GND_9), J9.16 (GND_10), J9.17 (GND_11), J9.4 (GND_1), J9.8 (GND_2), J9.9 (GND_3), Q4.E, Q5.E
- net SIM_VDD: now also J9.1 (VCC)
- net UART1_RXD: now also Q2.E
- net UART1_TXD: now also Q3.C
- net at C26.2, R20.1, U4.10 (UART1_RXD): now also Q2.C
- net at R27.2, R28.2: now also Q5.B
- net at R18.2: now also Q2.B
- net at D10.3 (K), R24.1: now also J9.3 (CLK)
- net at D10.4 (K), R26.2: now also J9.2 (RST)
- net at R19.2: now also Q3.B
- net at D10.1 (K), R23.1: now also J9.6 (I/O)
- net at R25.2: now also Q4.C
- net at U4.9 (UART1_TXD): now also Q3.E
- net at R29.2: now also Q5.C
- net at R21.2, R22.2: now also Q4.B
- no-connect marks 25 -> 26
Other:
- moved on the sheet: C32, D10, R23, R24, R26
