File: Enose_PCB/Enose_PCB.kicad_pcb (KiCad board)
At the start: 2 copper layers, 139 parts, among them IC1 ISL91127IRNZ-T7A, IC2 MP2722GRH-0000-Z, IC3 TPS22958DGNR, J1 Conn_01x04_Pin, J10 Fan, J2 Conn_01x04_Pin, J3 Conn_01x04_Pin, J4 DA15_Pins, J5 USB_C_Receptacle_USB2.0_16P, J6 Battery Terminal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

Commit message: Working on Enose PCB Layout
Parts:
- added C42: 100nF, Capacitor_SMD:C_0805_2012Metric_Pad1.18x1.45mm_HandSolder, F.Cu at (37.0, 93.5)
- added F1: Fuse Holder, SamacSys_Parts:64600001223, F.Cu at (71.5, 158.2)
- added TH1: Thermistor_NTC (10k), Connector_JST:JST_XH_B2B-XH-AM_1x02_P2.50mm_Vertical, F.Cu at (38.5, 85.0)
- added TP7: TestPoint, TestPoint:TestPoint_Pad_1.5x1.5mm, F.Cu at (85.2, 116.2)
- moved Q6 209.3 mm to (142.8, 248.0)
- moved C33 194.5 mm to (213.5, 246.5)
- moved C34 194.5 mm to (213.5, 249.5)
- moved C35 194.5 mm to (213.5, 252.5)
- moved J10 172.9 mm to (143.0, 237.0)
- moved C25 170.4 mm to (135.8, 256.8)
- moved D15 168.8 mm to (118.0, 241.9)
- moved R30 168.8 mm to (128.3, 254.6)
- moved R34 168.8 mm to (132.8, 245.8)
- moved C41 142.2 mm to (31.7, 123.8), turned to -90 degrees
- moved J1 139.3 mm to (241.2, 241.9)
- moved J2 139.3 mm to (227.0, 242.0)
- moved J3 139.3 mm to (230.8, 251.9)
- moved SW3 138.5 mm to (47.0, 126.8)
- moved TP3 135.5 mm to (42.0, 93.2)
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Connections:
- C11 pad 1: +BATT -> +SYS_SW
- C12 pad 1: +BATT -> +SYS_SW
- C17 pad 1: VBUS -> +VBUS
- C18 pad 2: VBUS -> +VBUS
- C24 pad 2: /Power Components/BATT -> +BATT
- C26 pad 2: Net-(U4-UART1_RXD) -> Net-(Q2-C)
- C40 pad 2: +BATT -> +SYS_SW
- C7 pad 1: +BATT -> +SYS_SW
- D11 pad 1: +BATT -> +SYS_SW
- D12 pad 2: +BATT -> +SYS_SW
- D8 pad 1: +15V -> Net-(D8-A1)
- D9 pad 2: +BATT -> +SYS_SW
- FB1 pad 2: +BATT -> +SYS_SW
- IC1 pad 10: +BATT -> +SYS_SW
- IC1 pad 11: +BATT -> +SYS_SW
- IC1 pad 6: +BATT -> +SYS_SW
- IC1 pad 7: +BATT -> +SYS_SW
- IC1 pad 8: +BATT -> +SYS_SW
- IC1 pad 9: +BATT -> +SYS_SW
- IC2 pad 12: /Power Components/BATT -> +BATT
- IC2 pad 14: /Power Components/BATT -> +BATT
- IC2 pad 2: VBUS -> +VBUS
- IC3 pad 5: +BATT -> +SYS_SW
- IC3 pad 8: +BATT -> +SYS_SW
- J4 pad 15: +15V -> Net-(D8-A1)
- J4 pad 7: +15V -> Net-(D8-A1)
- J4 pad 8: +15V -> Net-(D8-A1)
- J5 pad A4: VBUS -> +VBUS
- J5 pad A9: VBUS -> +VBUS
- J5 pad B4: VBUS -> +VBUS
- J5 pad B9: VBUS -> +VBUS
- J6 pad 1: /Power Components/BATT -> +BATT
- L3 pad 1: +BATT -> +SYS_SW
- PS1 pad 7: +BATT -> +SYS_SW
- Q1 pad 1: (no net) -> Net-(Q1-B)
- Q1 pad 2: (no net) -> GND
- Q1 pad 3: (no net) -> Net-(Q1-C)
- Q2 pad 1: (no net) -> Net-(Q2-B)
- Q2 pad 2: (no net) -> UART1_RXD
- Q2 pad 3: (no net) -> Net-(Q2-C)
- Q3 pad 1: (no net) -> Net-(Q3-B)
- Q3 pad 2: (no net) -> Net-(Q3-E)
- Q3 pad 3: (no net) -> UART1_TXD
- Q4 pad 1: (no net) -> Net-(Q4-B)
- Q4 pad 2: (no net) -> GND
- Q4 pad 3: (no net) -> Net-(Q4-C)
- Q5 pad 1: (no net) -> Net-(Q5-B)
- Q5 pad 2: (no net) -> GND
- Q5 pad 3: (no net) -> Net-(Q5-C)
- R16 pad 2: Net-(Q1-PadB) -> Net-(Q1-B)
- R17 pad 2: Net-(Q1-PadB) -> Net-(Q1-B)
- R18 pad 2: Net-(Q2-PadB) -> Net-(Q2-B)
- R19 pad 2: Net-(Q3-PadB) -> Net-(Q3-B)
- R20 pad 1: Net-(U4-UART1_RXD) -> Net-(Q2-C)
- R21 pad 2: Net-(Q4-PadB) -> Net-(Q4-B)
- R22 pad 2: Net-(Q4-PadB) -> Net-(Q4-B)
- R25 pad 2: Net-(Q4-PadC) -> Net-(Q4-C)
- R27 pad 2: Net-(Q5-PadB) -> Net-(Q5-B)
- R28 pad 2: Net-(Q5-PadB) -> Net-(Q5-B)
- R29 pad 2: Net-(Q5-PadC) -> Net-(Q5-C)
- R7 pad 1: +SYS -> +SYS_SW
- U2 pad 5: VBUS -> +VBUS
- U4 pad 1: Net-(U4-PWRKEY) -> Net-(Q1-C)
- U4 pad 10: Net-(U4-UART1_RXD) -> Net-(Q2-C)
- U4 pad 9: Net-(U4-UART1_TXD) -> Net-(Q3-E)
Routing:
- net +SYS_SW: track 0.00 -> 47.7 mm
- net Net-(U4-VBAT): track 0.00 -> 41.1 mm
- net +15V: track 0.00 -> 35.1 mm
- net +SYS: track 0.00 -> 29.5 mm
- net +VBUS: track 0.00 -> 18.8 mm
- net /Cellular Module/NETLIGHT: track 0.00 -> 12.9 mm
- net GND: track 0.00 -> 8.51 mm
- net /Cellular Module/RF_ANT: track 0.00 -> 7.56 mm
- net /Cellular Module/GNSS_ANT: track 0.00 -> 6.71 mm
- net Net-(PS1-COMP): track 0.00 -> 6.29 mm
- net Net-(PS1-FB): track 0.00 -> 6.19 mm
- net Net-(Q2-C): track 0.00 -> 5.71 mm
- net Net-(Q1-B): track 0.00 -> 5.17 mm
- net Net-(PS1-VCC): track 0.00 -> 5.09 mm
- net Net-(Q3-B): track 0.00 -> 3.08 mm
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
Commit message: Finished placeing components for Enose PCB
Parts:
- added H1: MountingHole, MountingHole:MountingHole_2.5mm, F.Cu at (80.0, 55.0)
- added H2: MountingHole, MountingHole:MountingHole_2.5mm, F.Cu at (190.0, 61.0)
- added H3: MountingHole, MountingHole:MountingHole_2.5mm, F.Cu at (80.0, 145.0)
- added H4: MountingHole, MountingHole:MountingHole_2.5mm, F.Cu at (190.0, 145.0)
- moved J3 242.1 mm to (88.8, 55.8), turned to -90 degrees
- moved J1 235.7 mm to (96.8, 55.7), turned to 0 degrees
- moved J2 222.4 mm to (105.5, 55.8), turned to -90 degrees
- moved C34 219.8 mm to (90.0, 67.8)
- moved C35 218.9 mm to (97.7, 66.8)
- moved C33 208.4 mm to (106.0, 68.0)
- moved C25 191.2 mm to (114.7, 66.8), turned to 90 degrees
- moved R30 190.7 mm to (121.9, 64.0), turned to 90 degrees
- moved D15 188.8 mm to (116.9, 53.0), turned to 180 degrees
- moved Q6 185.0 mm to (118.2, 64.7), turned to 90 degrees
- moved J10 180.1 mm to (118.2, 58.6), turned to 180 degrees
- moved R34 177.8 mm to (122.0, 68.3), turned to -90 degrees
- moved R5 80.9 mm to (173.5, 65.0)
- moved R4 80.8 mm to (173.5, 61.9)
- moved D1 77.5 mm to (178.2, 61.9)
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Connections:
- R31 pad 1: I2C_SCL -> ~{INT}
- R33 pad 1: ~{INT} -> I2C_SCL
- R35 pad 1: /PWM1 -> /PWM8
- R36 pad 1: /PWM2 -> /PWM7
- R37 pad 1: /PWM3 -> /PWM6
- R38 pad 1: /PWM4 -> /PWM5
- R39 pad 1: /PWM5 -> /PWM4
- R40 pad 1: /PWM6 -> /PWM3
- R41 pad 1: /PWM7 -> /PWM2
- R42 pad 1: /PWM8 -> /PWM1
- U1 pad 12: /Fan PWM -> unconnected-(U1-IO8-Pad12)
- U1 pad 15: Net-(SW2-B) -> unconnected-(U1-IO3-Pad15)
- U1 pad 23: unconnected-(U1-IO21-Pad23) -> /PWM7
- U1 pad 24: unconnected-(U1-IO47-Pad24) -> /PWM8
- U1 pad 25: unconnected-(U1-IO48-Pad25) -> Net-(SW2-B)
- U1 pad 27: I2C_SCL -> unconnected-(U1-IO0-Pad27)
- U1 pad 31: unconnected-(U1-IO38-Pad31) -> ~{INT}
- U1 pad 34: unconnected-(U1-IO41-Pad34) -> /ESP_LED1
- U1 pad 35: unconnected-(U1-IO42-Pad35) -> /ESP_LED2
- U1 pad 38: ~{INT} -> I2C_SCL
- U1 pad 6: /ESP_LED1 -> unconnected-(U1-IO6-Pad6)
- U1 pad 7: /ESP_LED2 -> unconnected-(U1-IO7-Pad7)
- U1 pad 8: /PWM7 -> unconnected-(U1-IO15-Pad8)
- U1 pad 9: /PWM8 -> /Fan PWM
Routing:
- net USB_D-: track 2.44 -> 76.8 mm
- net USB_D+: track 2.44 -> 74.0 mm
- net +SYS_SW: track 47.7 -> 0.00 mm
- net +15V: track 35.1 -> 13.8 mm
- net +VBUS: track 18.8 -> 0.00 mm
- net I2C_SCL: track 0.00 -> 17.0 mm
- net I2C_SDA: track 0.00 -> 17.0 mm
- net /Cellular Module/NETLIGHT: track 12.9 -> 2.16 mm
- net +SYS: track 29.5 -> 23.2 mm
- net Net-(U4-VBAT): track 41.1 -> 35.2 mm
Other:
- board outline added: 120 x 100 mm

Commit message: Added so netlabels
Parts:
- moved J5 16.3 mm to (78.7, 73.5)
- moved SW3 16.0 mm to (106.5, 112.0)
- moved SW4 13.5 mm to (77.2, 88.2)
- moved J9 5.72 mm to (176.0, 82.0)
- moved SW2 4.98 mm to (154.2, 82.0), turned to 0 degrees
- moved U2 4.58 mm to (89.0, 77.5), turned to 90 degrees
- moved D5 4.47 mm to (130.0, 142.2), turned to 0 degrees
- moved D11 4.26 mm to (151.5, 127.5), turned to 0 degrees
- moved D16 3.51 mm to (95.8, 115.3)
- moved R9 3.10 mm to (130.0, 139.8)
- moved R31 0.54 mm to (167.0, 67.2)
- moved TP4 0.54 mm to (130.8, 135.2)
- moved J7 0.14 mm to (164.3, 129.8)
- moved D13 0.06 mm to (179.7, 130.1)
- turned C11 to 180 degrees
Routing:
- net +SYS: track 23.2 -> 0.00 mm
- net +15V: track 13.8 -> 32.5 mm
- net Net-(D16-K7): track 0.00 -> 18.7 mm
- net Net-(D16-K5): track 0.00 -> 18.4 mm
- net Net-(D16-K3): track 0.00 -> 18.1 mm
- net Net-(D16-K1): track 0.00 -> 17.8 mm
- net Net-(D16-K8): track 0.00 -> 17.5 mm
- net Net-(D16-K6): track 0.00 -> 17.1 mm
- net Net-(D16-K4): track 0.00 -> 16.9 mm
- net Net-(D16-K2): track 0.00 -> 16.5 mm
- net USB_D-: track 76.8 -> 62.4 mm
- net USB_D+: track 74.0 -> 61.6 mm
- net Net-(U4-VBAT): track 35.2 -> 41.3 mm
- net GND: track 8.51 -> 10.8 mm
- net Net-(IC3-CT): track 0.00 -> 1.57 mm
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- added copper zone on F.Cu, net +15V
- added copper zone on F.Cu, net +SYS_SW
- added copper zone on B.Cu, net GND
