File: Enose_PCB/Enose_PCB_2_Layer.kicad_pcb (KiCad board)
At the start: 2 copper layers, 120 x 100 mm, 147 parts, among them IC1 ISL91127IRNZ-T7A, IC2 MP2722GRH-0000-Z, IC3 TPS22958DGNR, J1 Conn_01x04_Pin, J10 Fan, J2 Conn_01x04_Pin, J3 Conn_01x04_Pin, J4 DA15_Pins, J5 USB_C_Receptacle_USB2.0_16P, J6 Battery Terminal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

Commit message: Enose PCB almost done
Parts:
- moved R17 55.3 mm to (154.8, 112.0)
- moved Q1 55.3 mm to (158.4, 112.0)
- moved R16 51.5 mm to (155.8, 108.5), turned to 180 degrees
- moved R25 41.2 mm to (177.8, 143.5)
- moved D3 40.1 mm to (117.0, 112.3), turned to 180 degrees
- moved D9 37.5 mm to (174.2, 142.3), turned to 90 degrees
- moved R22 36.6 mm to (182.5, 141.7), turned to 90 degrees
- moved Q4 35.3 mm to (178.8, 139.5), turned to -90 degrees
- moved R7 35.0 mm to (117.0, 109.8)
- moved R31 32.2 mm to (167.0, 67.2), turned to 0 degrees
- moved R32 32.2 mm to (167.2, 58.4)
- moved R33 32.0 mm to (167.2, 61.3), turned to 0 degrees
- moved R21 30.1 mm to (182.5, 137.5), turned to -90 degrees
- moved C33 14.2 mm to (106.0, 68.0), turned to 0 degrees
- moved C34 13.7 mm to (90.0, 67.8), turned to 0 degrees
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Connections:
- net /Power Components/LX1 renamed Net-(IC1-LX1_1)
- net /Power Components/LX2 renamed Net-(IC1-LX2_1)
- J1 pad 1: +3V3 -> I2C_SDA
- J1 pad 2: GND -> I2C_SCL
- J1 pad 3: I2C_SDA -> GND
- J1 pad 4: I2C_SCL -> +3V3
- J2 pad 1: +3V3 -> I2C_SDA
- J2 pad 2: GND -> I2C_SCL
- J2 pad 3: I2C_SDA -> GND
- J2 pad 4: I2C_SCL -> +3V3
- J3 pad 1: +3V3 -> I2C_SDA
- J3 pad 2: GND -> I2C_SCL
- J3 pad 3: I2C_SDA -> GND
- J3 pad 4: I2C_SCL -> +3V3
- Q2 pad 2: UART1_TXD -> UART1_RXD
- Q3 pad 3: UART1_RXD -> UART1_TXD
- R2 pad 2: UART1_RXD -> UART1_TXD
- U1 pad 10: ~{INT} -> PWRKEY
- U1 pad 11: I2C_SDA -> EN(15V)
- U1 pad 12: I2C_SCL -> unconnected-(U1-IO8-Pad12)
- U1 pad 25: unconnected-(U1-IO48-Pad25) -> Net-(SW2-B)
- U1 pad 27: Net-(SW2-B) -> unconnected-(U1-IO0-Pad27)
- U1 pad 31: unconnected-(U1-IO38-Pad31) -> ~{INT}
- U1 pad 36: UART1_RXD -> UART1_TXD
- U1 pad 37: UART1_TXD -> UART1_RXD
- U1 pad 38: unconnected-(U1-IO2-Pad38) -> I2C_SCL
- U1 pad 39: PWRKEY -> I2C_SDA
- U1 pad 8: EN(15V) -> unconnected-(U1-IO15-Pad8)
Routing:
- net +3V3: track 134.7 -> 0.00 mm, vias 2 -> 0
- net /PWM8: track 121.4 -> 0.00 mm, vias 2 -> 0
- net /PWM6: track 120.5 -> 0.00 mm, vias 2 -> 0
- net /PWM2: track 120.4 -> 0.00 mm, vias 2 -> 0
- net /PWM4: track 119.8 -> 0.00 mm, vias 2 -> 0
- net /PWM7: track 116.9 -> 0.00 mm, vias 2 -> 0
- net /PWM1: track 116.4 -> 0.00 mm, vias 2 -> 0
- net /PWM5: track 115.9 -> 0.00 mm, vias 2 -> 0
- net /PWM3: track 115.8 -> 0.00 mm, vias 2 -> 0
- net +SYS_SW: track 98.4 -> 0.00 mm
- net I2C_SDA: track 96.2 -> 17.0 mm, vias 4 -> 0
- net I2C_SCL: track 89.8 -> 17.0 mm, vias 4 -> 0
- net Net-(Q1-C): track 72.5 -> 0.00 mm
- net EN(15V): track 70.3 -> 0.00 mm, vias 4 -> 0
- net Net-(IC3-ON): track 66.6 -> 0.00 mm, vias 4 -> 0
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- removed copper zone on F.Cu, net +BATT
- removed copper zone on F.Cu, net +SYS
- removed copper zone on F.Cu, net +VBUS
- removed copper zone on F.Cu, net Net-(IC1-LX1_1)
- removed copper zone on F.Cu, net Net-(IC1-LX2_1)
Other:
- outline, holes or cut-outs redrawn
