File: Multi-emitter V2 Thesis/Multi-emitter V2 Thesis.kicad_sch (KiCad schematic)
At the start: 44 parts, among them J1 Emitter0 Input, J2 Emitter4 Input, J3 Emitter1 Input, J4 Emitter5 Input, J5 Emitter2 Input, J6 Emitter6 Input, J8 Emitter3 Input, J9 Emitter7 Input, Q1 NMOS, Q2 NMOS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

Commit message: testing comment change on pcb to play with git pushing
Other:
- note added: "TODO: 1. Add 200-300 Ohm resistor to gates for ESD protection (see recomended values) 2. Add D-sub port with added ESD protection IC on input 3. Add input protection on the mosfet input 4. See if mosfet needs a protection diode."
Changed lines of the file:
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@@
+		)
+	)
+	(text "TODO:\n1. Add 200-300 Ohm resistor to gates for ESD protection (see recomended values)\n2. Add D-sub port with added ESD protection IC on input\n3. Add input protection on the mosfet input\n4. See if mosfet needs a protection diode."
+		(exclude_from_sim no)
+		(at 100.584 139.192 0)
+		(effects
+			(font
+				(size 1.27 1.27)
+			)
+			(justify left)
 		)
 	)

Commit message: pushing some changes only a bit to go
Parts:
- removed C2, C3, C4, C5, C6, C7, C8: 100n, Capacitor_THT:C_Disc_D5.0mm_W2.5mm_P5.00mm, symbol Device:C
- removed J2: Emitter4 Input, TerminalBlock:TerminalBlock_bornier-2_P5.08mm, symbol Connector:Screw_Terminal_01x02
- removed J3: Emitter1 Input, TerminalBlock:TerminalBlock_bornier-2_P5.08mm, symbol Connector:Screw_Terminal_01x02
- removed J4: Emitter5 Input, TerminalBlock:TerminalBlock_bornier-2_P5.08mm, symbol Connector:Screw_Terminal_01x02
- removed J5: Emitter2 Input, TerminalBlock:TerminalBlock_bornier-2_P5.08mm, symbol Connector:Screw_Terminal_01x02
- removed J8: Emitter3 Input, TerminalBlock:TerminalBlock_bornier-2_P5.08mm, symbol Connector:Screw_Terminal_01x02
- removed J9: Emitter7 Input, TerminalBlock:TerminalBlock_bornier-2_P5.08mm, symbol Connector:Screw_Terminal_01x02
- removed L2, L3, L4, L5, L6, L7, L8: 220u, Inductor_THT:L_Radial_D7.2mm_P3.00mm_Murata_1700, symbol Device:L
- removed Q2, Q3, Q4, Q5, Q6, Q7, Q8: NMOS, Package_DIP:Vishay_HVM-DIP-3_W7.62mm, symbol Simulation_SPICE:NMOS
- removed R2, R3, R5, R6, R7, R8: 10k, Resistor_THT:R_Axial_DIN0207_L6.3mm_D2.5mm_P10.16mm_Horizontal, symbol Device:R
- removed R4: 10k, symbol Device:R
- added D1: DT1240A-08LP3810, Package_DFN_QFN:UDFN-9_1.0x3.8mm_P0.5mm, symbol Power_Protection:DT1240A-08LP3810
- added J?: DA15_Pins, KiCad:XM3B1522112, symbol Connector:DA15_Pins
Connections:
- net PWM0 is gone; now on net PWM1: Q1.2 (G), R1.1
- net GND: now also D1.3 (A), J?.13 (P13), J?.14 (P14), J?.5, J?.6
- net PWM1: now also D1.1 (K1), J?.12 (P12)
- net PWM2: now also D1.2 (K2), J?.4
- net PWM3: now also D1.4 (K3), J?.11 (P111)
- net PWM4: now also D1.5 (K4), J?.3
- net PWM5: now also D1.6 (K5), J?.10 (P10)
- net PWM6: now also D1.7 (K6), J?.2
- net PWM7: now also D1.8 (K7), J?.9 (P9)
- net VCC: now also J?.15 (P15), J?.7, J?.8
- new net PWM8: D1.9 (K8), J?.1
Other:
- note added: "Notes: 1.PWM inputs typical signal behaviour is either off state or 100-115 kHz. 2.VCC should be between 13-16V."
- note added: "TODO: 1. Verify if the DT1240A-08LP3810Q is a good ESD IC 2. Add 2-pin JST connectors to match the emitter JST so they can easily be plugged in without havign to modify the wire ends. flyback diode on input filter not needed as currents are very low 3. Add a fuse to protect mosfet short circuit event (can happen if PWM inputs are either DC high or are driving at very high frequency) 4. Change som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"
- note removed: "TODO: 1. Add 200-300 Ohm resistor to gates for ESD protection (see recomended values) 2. Add D-sub port with added ESD protection IC on input 3. Add input protection on the mosfet input 4. See if mosfet needs a protection diode."
